Commit message: Implement gripper action
1. Separate gripper base and mover
. Modify URDF files and and add joint6
. Add gripper action into chase_moveit.py
2. Add 2 place position
3. Remove parking, then just stay at last position
4. Add print angles for inits.yaml, rebearm_description.urdf.xacro range

File: rebearm_description/xacro/rebearm.ros2_control.xacro (robot description, xacro)
@@ -37,4 +37,18 @@
         <state_interface name="position"/>
       </joint>
+      <joint name="${prefix}joint5">
+        <command_interface name="position">
+          <param name="min">-1</param>
+          <param name="max">1</param>
+        </command_interface>
+        <state_interface name="position"/>
+      </joint>
+      <joint name="${prefix}joint6">
+        <command_interface name="position">
+          <param name="min">-1</param>
+          <param name="max">1</param>
+        </command_interface>
+        <state_interface name="position"/>
+      </joint>
     </ros2_control>
   </xacro:macro>

File: rebearm_description/xacro/rebearm_description.urdf.xacro (robot description, xacro)
@@ -45,7 +45,15 @@
   <xacro:property name="width5"    value="0.045" />  <!-- Square dimensions (widthxwidth) -->
   <xacro:property name="height5"   value="0.95" />   <!-- Link 5, blue -->
-  <xacro:property name="offsetx45" value="-0.120" />  <!-- Link position from previous link -->
+  <xacro:property name="offsetx45" value="-0.120" /> <!-- Link position from previous link -->
   <xacro:property name="offsety45" value="-0.230" />
   <xacro:property name="offsetz45" value="0.020" />
+  <xacro:property name="offsetx6"  value="0.000" />  <!-- joint6 location x,y,z on link5-->
+  <xacro:property name="offsety6"  value="-0.120" />
+  <xacro:property name="offsetz6"  value="0.195" />
+  <xacro:property name="width6"    value="0.045" />  <!-- Square dimensions (widthxwidth) -->
+  <xacro:property name="height6"   value="0.95" />   <!-- Link 6, blue -->
+  <xacro:property name="offsetx56" value="-0.120" /> <!-- Link position from previous link -->
+  <xacro:property name="offsety56" value="-0.180" />
+  <xacro:property name="offsetz56" value="-0.180" />
   <xacro:property name="axel_offset" value="0.0" />  <!-- Space btw top of beam and the each joint -->
   <!-- Base Link -->
@@ -77,5 +85,5 @@
     <axis xyz="0 0 1"/>
     <dynamics damping="0.7"/>
-    <limit velocity="4.8" effort="1" lower="${-pi*0.33}" upper="${pi*0.33}" />
+    <limit velocity="4.8" effort="1" lower="-1.57" upper="1.57" />
   </joint>
   <!-- Link 1-->
@@ -110,5 +118,5 @@
     <filename xyz="-1 0 0"/>
     <dynamics damping="0.7"/>
-    <limit velocity="4.8" effort="1" lower="${-pi}" upper="${pi}" />
+    <limit velocity="4.8" effort="1" lower="0.52" upper="-0.105" />
   </joint>
   <!-- Link 2-->
@@ -143,5 +151,5 @@
     <axis xyz="1 0 0"/>
     <dynamics damping="0.7"/>
-    <limit velocity="4.8" effort="1" lower="${-pi}" upper="${pi}" />
+    <limit velocity="4.8" effort="1" lower="-0.78" upper="-2.09" />
   </joint>
   <!-- Link 3 -->
@@ -176,5 +184,5 @@
     <axis xyz="1 0 0"/>
     <dynamics damping="0.7"/>
-    <limit velocity="4.8" effort="1" lower="${-pi}" upper="${pi}" />
+    <limit velocity="4.8" effort="1" lower="-0.87" upper="-2.09" />
   </joint>
   <!-- Link 4 -->
@@ -209,7 +217,7 @@
     <axis xyz="0 0 1"/>
     <dynamics damping="0.7"/>
-    <limit velocity="4.8" effort="1" lower="${-pi}" upper="${pi}" />
-  </joint>
-  <!-- Link 5, gripper -->
+    <limit velocity="4.8" effort="1" lower="0.0" upper="${-pi*0.5}" />
+  </joint>
+  <!-- Link 5, gripper base -->
   <link name="${prefix}link5">
   <collision>
@@ -235,4 +243,37 @@
     </inertial>
   </link>
+  <!-- Joint 6, z origin = parent height  -->
+    <joint name="${prefix}joint6" type="revolute">
+    <origin xyz="${offsetx6} ${offsety6} ${offsetz6}" rpy="0.0 0.0 0.0"/>
+    <parent link="${prefix}link5"/>
+    <child link="${prefix}link6" />
+    <axis xyz="1 0 0"/>
+    <dynamics damping="0.7"/>
+    <limit velocity="4.8" effort="1" lower="-1.40" upper="-1.00" />
+  </joint>
+  <!-- Link 6, gripper mover -->
+  <link name="${prefix}link6">
+  <collision>
+    <origin xyz="${offsetx56} ${offsety56} ${offsetz56}" rpy="0.0 0.0 0.0"/>
+    <geometry>
+      <box size="${width5} ${width5} ${height5}"/>
+    </geometry>
+  </collision>
+  <visual>
+    <origin xyz="${offsetx56} ${offsety56} ${offsetz56}" rpy="0 0.0 0.0 "/>
+    <geometry>
+      <mesh filename="package://rebearm_description/meshes/URDF_joint6.stl" scale="0.005 0.005 0.005" />
+    </geometry>
+    <material name="blue"/>
+  </visual>
+  <inertial>
+    <origin xyz="0 0 0" rpy="0.0 0.0 0.0"/>
+    <mass value="${mass}"/>
+    <inertia
+      ixx="${mass / 12.0 * (width4*width4 + height4*height4)}" ixy="0.0" ixz="0.0"
+      iyy="${mass / 12.0 * (height4*height4 + width4*width4)}" iyz="0.0"
+      izz="${mass / 12.0 * (width4*width4 + width4*width4)}"/>
+    </inertial>
+  </link>
   </xacro:macro>
 </robot>
