Commit message: Fix wrong direction of joint6

File: rebearm_description/xacro/rebearm_description.urdf.xacro (robot description, xacro)
@@ -46,14 +46,14 @@
   <xacro:property name="height5"   value="0.95" />   <!-- Link 5, blue -->
   <xacro:property name="offsetx45" value="-0.120" /> <!-- Link position from previous link -->
-  <xacro:property name="offsety45" value="-0.230" />
-  <xacro:property name="offsetz45" value="0.020" />
+  <xacro:property name="offsety45" value="-0.166" />
+  <xacro:property name="offsetz45" value="0.000" />
   <xacro:property name="offsetx6"  value="0.000" />  <!-- joint6 location x,y,z on link5-->
-  <xacro:property name="offsety6"  value="-0.120" />
-  <xacro:property name="offsetz6"  value="0.195" />
+  <xacro:property name="offsety6"  value="-0.07" />
+  <xacro:property name="offsetz6"  value="0.178" />
   <xacro:property name="width6"    value="0.045" />  <!-- Square dimensions (widthxwidth) -->
   <xacro:property name="height6"   value="0.95" />   <!-- Link 6, blue -->
   <xacro:property name="offsetx56" value="-0.120" /> <!-- Link position from previous link -->
-  <xacro:property name="offsety56" value="-0.180" />
-  <xacro:property name="offsetz56" value="-0.180" />
+  <xacro:property name="offsety56" value="0.053" />
+  <xacro:property name="offsetz56" value="-0.050" />
   <xacro:property name="axel_offset" value="0.0" />  <!-- Space btw top of beam and the each joint -->
   <!-- Base Link -->
@@ -217,5 +217,5 @@
     <axis xyz="0 0 1"/>
     <dynamics damping="0.7"/>
-    <limit velocity="4.8" effort="1" lower="0.0" upper="${-pi*0.5}" />
+    <limit velocity="4.8" effort="1" lower="${pi*0.5}" upper="${-pi*0.5}" />
   </joint>
   <!-- Link 5, gripper base -->
@@ -250,10 +250,10 @@
     <axis xyz="1 0 0"/>
     <dynamics damping="0.7"/>
-    <limit velocity="4.8" effort="1" lower="-1.40" upper="-1.00" />
+  <limit velocity="-4.8" effort="1" lower="-1.6" upper="-1.04" />
   </joint>
   <!-- Link 6, gripper mover -->
   <link name="${prefix}link6">
   <collision>
-    <origin xyz="${offsetx56} ${offsety56} ${offsetz56}" rpy="0.0 0.0 0.0"/>
+    <origin xyz="${offsetx56} ${offsety56} ${offsetz56}" rpy="${pi*0.5} 0.0 0.0"/>
     <geometry>
       <box size="${width5} ${width5} ${height5}"/>
@@ -261,5 +261,5 @@
   </collision>
   <visual>
-    <origin xyz="${offsetx56} ${offsety56} ${offsetz56}" rpy="0 0.0 0.0 "/>
+    <origin xyz="${offsetx56} ${offsety56} ${offsetz56}" rpy="${pi*0.5} 0.0 0.0"/>
     <geometry>
       <mesh filename="package://rebearm_description/meshes/URDF_joint6.stl" scale="0.005 0.005 0.005" />

Commit message: Add cube marker
1. Add cube marker in rebearm_description
2. Delete rebearm_bringup folder
3. Delete CMakeLists.txt which are not used
4. version string set to 0.9.1
5. Add gripper calibration

File: rebearm_description/xacro/rebearm_description.urdf.xacro (robot description, xacro)
@@ -250,5 +250,5 @@
     <axis xyz="1 0 0"/>
     <dynamics damping="0.7"/>
-  <limit velocity="-4.8" effort="1" lower="-1.6" upper="-1.04" />
+  <limit velocity="4.8" effort="1" lower="-1.6" upper="-1.04" />
   </joint>
   <!-- Link 6, gripper mover -->
